Commit message: More advances

File: setup_description/urdf/robot.urdf.xacro (robot description, xacro)
@@ -43,5 +43,5 @@
     input_recipe_filename="$(arg input_recipe_filename)"
   >
-    <origin xyz="0 0 0" rpy="0 0 0" />          <!-- position robot in the world -->
+    <origin xyz="0 0 0" rpy="0 0 0" />
   </xacro:ur_robot>
   <xacro:ur_to_robotiq prefix="" parent="tool0" child="adapter_to_gripper"/>
@@ -53,5 +53,5 @@
     use_fake_hardware="$(arg use_fake_hardware)"
     com_port="$(arg gripper_com_port)">
-    <origin xyz="0 0 0.01" rpy="0 0 ${pi/2}"/>
+    <origin xyz="0 0 0" rpy="0 0 0"/>
   </xacro:robotiq_gripper>
   <!-- Virtual link for end effector at the fingertips -->
@@ -60,5 +60,5 @@
       <origin xyz="0 0 0" rpy="0 0 0"/>
       <geometry>
-        <sphere radius="0.001"/> <!-- invisible tiny sphere -->
+        <sphere radius="0.001"/>
       </geometry>
       <material name="transparent">

Commit message: Almost working

File: setup_description/urdf/robot.urdf.xacro (robot description, xacro)
@@ -23,4 +23,10 @@
   <xacro:arg name="output_recipe_filename" default=""/>
   <xacro:arg name="input_recipe_filename" default=""/>
+  <xacro:arg name="tool_voltage" default="24"/>
+  <xacro:arg name="tool_baudrate" default="115200"/>
+  <xacro:arg name="tool_parity" default="0" />
+  <xacro:arg name="tool_stop_bits" default="1" />
+  <xacro:arg name="tool_rx_idle_chars" default="1.5"/>
+  <xacro:arg name="tool_tx_idle_chars" default="3.5" />
   <!-- create link fixed to the "world" -->
   <link name="world" />
@@ -42,4 +48,10 @@
     output_recipe_filename="$(arg output_recipe_filename)"
     input_recipe_filename="$(arg input_recipe_filename)"
+    tool_voltage="$(arg tool_voltage)"
+    tool_baud_rate="$(arg tool_baudrate)"
+    tool_parity="$(arg tool_parity)"
+    tool_stop_bits="$(arg tool_stop_bits)"
+    tool_rx_idle_chars="$(arg tool_rx_idle_chars)"
+    tool_tx_idle_chars="$(arg tool_tx_idle_chars)"
   >
     <origin xyz="0 0 0" rpy="0 0 0" />
@@ -70,5 +82,5 @@
     <parent link="tool0"/>
     <child link="ee_link"/>
-    <origin xyz="0 0 0.22" rpy="0 0 0"/>
+    <origin xyz="0 0 0.12" rpy="0 0 0"/>
   </joint>
 </robot>

Commit message: Offset corrected

File: setup_description/urdf/robot.urdf.xacro (robot description, xacro)
@@ -82,5 +82,5 @@
     <parent link="tool0"/>
     <child link="ee_link"/>
-    <origin xyz="0 0 0.12" rpy="0 0 0"/>
+    <origin xyz="0 0 0.22" rpy="0 0 0"/>
   </joint>
 </robot>

Commit message: Camera added and dockerized

File: setup_description/urdf/robot.urdf.xacro (robot description, xacro)
@@ -5,4 +5,5 @@
   <xacro:include filename="$(find robotiq_description)/urdf/robotiq_2f_140_macro.urdf.xacro" />
   <xacro:include filename="$(find robotiq_description)/urdf/ur_to_robotiq_adapter.urdf.xacro" />
+  <xacro:include filename="$(find realsense2_description)/urdf/_d435.urdf.xacro" />
   <xacro:arg name="ur_type" default="ur10e"/>
   <!-- parameters -->
@@ -29,4 +30,7 @@
   <xacro:arg name="tool_rx_idle_chars" default="1.5"/>
   <xacro:arg name="tool_tx_idle_chars" default="3.5" />
+  <xacro:arg name="use_nominal_extrinsics" default="false"/>
+  <xacro:arg name="add_plug" default="false" />
+  <xacro:arg name="use_mesh" default="true" />
   <!-- create link fixed to the "world" -->
   <link name="world" />
@@ -84,3 +88,7 @@
     <origin xyz="0 0 0.22" rpy="0 0 0"/>
   </joint>
+  <!-- Realsense D435 Camera -->
+  <xacro:sensor_d435 parent="base_link" use_nominal_extrinsics="$(arg use_nominal_extrinsics)" add_plug="$(arg add_plug)" use_mesh="$(arg use_mesh)">
+    <origin xyz="0 0 1.0" rpy="0 0 0"/>
+  </xacro:sensor_d435>
 </robot>

Commit message: Added gazebo ignition, deleted useless control_node from ur_control.launch.py

File: setup_description/urdf/robot.urdf.xacro (robot description, xacro)
@@ -2,4 +2,5 @@
 <robot xmlns:xacro="http://wiki.ros.org/xacro" name="$(arg name)">
   <xacro:arg name="name" default="ur"/>
+  <xacro:arg name="use_sim" default="false"/>
   <xacro:include filename="$(find ur_description)/urdf/ur_macro.xacro"/>
   <xacro:include filename="$(find robotiq_description)/urdf/robotiq_2f_140_macro.urdf.xacro" />
@@ -29,4 +30,16 @@
   <xacro:arg name="tool_rx_idle_chars" default="1.5"/>
   <xacro:arg name="tool_tx_idle_chars" default="3.5" />
+  <xacro:arg name="controllers_file" default="config/ur_controllers.yaml"/>
+  <!-- Gazebo Ignition plugin -->
+  <xacro:property name="comparable_use_sim" value="$(arg use_sim)" />
+  <xacro:if value="${comparable_use_sim}">
+    <xacro:include filename="$(find setup_description)/gazebo/ur_robotiq.ignition_macro.xacro" />
+    <xacro:ur_robotiq_ignition_macro
+      runtime_config_package="setup_description"
+      path_to_yaml="$(arg controllers_file)"
+      namespace="/"
+      prefix="$(arg tf_prefix)"
+    />
+  </xacro:if>
   <!-- create link fixed to the "world" -->
   <link name="world" />
@@ -43,4 +56,5 @@
     safety_pos_margin="$(arg safety_pos_margin)"
     safety_k_position="$(arg safety_k_position)"
+    sim_ignition="$(arg use_sim)"
     use_tool_communication="$(arg use_tool_communication)"
     robot_ip="$(arg robot_ip)"
@@ -63,4 +77,5 @@
     prefix=""
     parent="adapter_to_gripper"
+    sim_ignition="$(arg use_sim)"
     use_fake_hardware="$(arg use_fake_hardware)"
     com_port="$(arg gripper_com_port)">

Commit message: Added camera flange support

File: setup_description/urdf/robot.urdf.xacro (robot description, xacro)
@@ -31,4 +31,5 @@
   <xacro:arg name="tool_tx_idle_chars" default="3.5" />
   <xacro:arg name="controllers_file" default="config/ur_controllers.yaml"/>
+  <xacro:arg name="use_cam_flange_support" default="false"/>
   <!-- Gazebo Ignition plugin -->
   <xacro:property name="comparable_use_sim" value="$(arg use_sim)" />
@@ -71,5 +72,17 @@
     <origin xyz="0 0 0" rpy="0 0 0" />
   </xacro:ur_robot>
-  <xacro:ur_to_robotiq prefix="" parent="tool0" child="adapter_to_gripper"/>
+  <!-- Camera flange support -->
+  <xacro:property name="comparable_use_cam_flange_support" value="$(arg use_cam_flange_support)" />
+  <xacro:if value="${comparable_use_cam_flange_support}">
+    <xacro:property name="ur_to_robotiq_adapter_parent" value="cam_flange_ring_mounting" />
+    <xacro:include filename="$(find cam_flange_support)/urdf/cam_flange_support_macro.urdf.xacro" />
+    <xacro:cam_flange_support parent="tool0" >
+      <origin xyz="0 0 0" rpy="0 0 ${pi}" />
+    </xacro:cam_flange_support>
+  </xacro:if>
+  <xacro:unless value="${comparable_use_cam_flange_support}">
+    <xacro:property name="ur_to_robotiq_adapter_parent" value="tool0" />
+  </xacro:unless>
+  <xacro:ur_to_robotiq prefix="" parent="${ur_to_robotiq_adapter_parent}" child="adapter_to_gripper"/>
   <!-- Robotiq 2F-140 Gripper connected to adapter -->
   <xacro:robotiq_gripper

File: setup_moveit_config/srdf/ur.srdf.xacro (robot description, xacro)
@@ -5,5 +5,6 @@
   <!-- parameters -->
   <xacro:arg name="prefix" default="" />
+  <xacro:arg name="use_cam_flange_support" default="false"/>
   <xacro:include filename="$(find setup_moveit_config)/srdf/ur_macro.srdf.xacro"/>
-  <xacro:ur_srdf name="$(arg name)" prefix="$(arg prefix)"/>
+  <xacro:ur_srdf name="$(arg name)" prefix="$(arg prefix)" use_cam_flange_support="$(arg use_cam_flange_support)"/>
 </robot>
