Commit message: Added camera flange support

File: setup_moveit_config/srdf/ur_macro.srdf.xacro (robot description, xacro)
@@ -5,5 +5,5 @@
     A URDF file must exist for this robot as well, where the joints and the links that are referenced are defined
 -->
-  <xacro:macro name="ur_srdf" params="name prefix">
+  <xacro:macro name="ur_srdf" params="name prefix use_cam_flange_support">
     <!--GROUPS - Representation of a set of joints and links. This can be useful for specifying DOF to plan for, defining arms, end effectors, etc-->
     <!--LINKS - When a link is specified, the parent joint of that link (if it exists) is automatically included-->
@@ -65,117 +65,125 @@
       type="fixed"
       parent_frame="world"
-      child_link="base_link"/>
+      child_link="${prefix}base_link"/>
     <!--DISABLE COLLISIONS - By default it is assumed that any link of the robot could potentially come into collision with any other link in the robot. This tag disables collision checking between a specified pair of links. -->
-    <disable_collisions link1="base_link_inertia" link2="shoulder_link" reason="Adjacent"/>
-    <disable_collisions link1="base_link_inertia" link2="upper_arm_link" reason="Never"/>
-    <disable_collisions link1="base_link_inertia" link2="wrist_1_link" reason="Never"/>
-    <disable_collisions link1="forearm_link" link2="upper_arm_link" reason="Adjacent"/>
-    <disable_collisions link1="forearm_link" link2="wrist_1_link" reason="Adjacent"/>
-    <disable_collisions link1="left_inner_finger" link2="left_inner_finger_pad" reason="Adjacent"/>
-    <disable_collisions link1="left_inner_finger" link2="left_inner_knuckle" reason="Default"/>
-    <disable_collisions link1="left_inner_finger" link2="left_outer_finger" reason="Adjacent"/>
-    <disable_collisions link1="left_inner_finger" link2="left_outer_knuckle" reason="Never"/>
-    <disable_collisions link1="left_inner_finger" link2="right_inner_finger" reason="Never"/>
-    <disable_collisions link1="left_inner_finger" link2="right_inner_finger_pad" reason="Never"/>
-    <disable_collisions link1="left_inner_finger" link2="right_inner_knuckle" reason="Never"/>
-    <disable_collisions link1="left_inner_finger" link2="right_outer_finger" reason="Never"/>
-    <disable_collisions link1="left_inner_finger" link2="right_outer_knuckle" reason="Never"/>
-    <disable_collisions link1="left_inner_finger" link2="robotiq_140_base_link" reason="Never"/>
-    <disable_collisions link1="left_inner_finger" link2="ur_to_robotiq_link" reason="Never"/>
-    <disable_collisions link1="left_inner_finger" link2="wrist_1_link" reason="Never"/>
-    <disable_collisions link1="left_inner_finger" link2="wrist_2_link" reason="Never"/>
-    <disable_collisions link1="left_inner_finger" link2="wrist_3_link" reason="Never"/>
-    <disable_collisions link1="left_inner_finger_pad" link2="left_inner_knuckle" reason="Never"/>
-    <disable_collisions link1="left_inner_finger_pad" link2="left_outer_finger" reason="Never"/>
-    <disable_collisions link1="left_inner_finger_pad" link2="left_outer_knuckle" reason="Never"/>
-    <disable_collisions link1="left_inner_finger_pad" link2="right_inner_finger" reason="Never"/>
-    <disable_collisions link1="left_inner_finger_pad" link2="right_inner_knuckle" reason="Never"/>
-    <disable_collisions link1="left_inner_finger_pad" link2="right_outer_finger" reason="Never"/>
-    <disable_collisions link1="left_inner_finger_pad" link2="right_outer_knuckle" reason="Never"/>
-    <disable_collisions link1="left_inner_finger_pad" link2="robotiq_140_base_link" reason="Never"/>
-    <disable_collisions link1="left_inner_finger_pad" link2="ur_to_robotiq_link" reason="Never"/>
-    <disable_collisions link1="left_inner_finger_pad" link2="wrist_1_link" reason="Never"/>
-    <disable_collisions link1="left_inner_finger_pad" link2="wrist_2_link" reason="Never"/>
-    <disable_collisions link1="left_inner_finger_pad" link2="wrist_3_link" reason="Never"/>
-    <disable_collisions link1="left_inner_knuckle" link2="left_outer_finger" reason="Never"/>
-    <disable_collisions link1="left_inner_knuckle" link2="left_outer_knuckle" reason="Default"/>
-    <disable_collisions link1="left_inner_knuckle" link2="right_inner_finger" reason="Never"/>
-    <disable_collisions link1="left_inner_knuckle" link2="right_inner_finger_pad" reason="Never"/>
-    <disable_collisions link1="left_inner_knuckle" link2="right_inner_knuckle" reason="Never"/>
-    <disable_collisions link1="left_inner_knuckle" link2="right_outer_finger" reason="Never"/>
-    <disable_collisions link1="left_inner_knuckle" link2="right_outer_knuckle" reason="Never"/>
-    <disable_collisions link1="left_inner_knuckle" link2="robotiq_140_base_link" reason="Adjacent"/>
-    <disable_collisions link1="left_inner_knuckle" link2="ur_to_robotiq_link" reason="Never"/>
-    <disable_collisions link1="left_inner_knuckle" link2="wrist_1_link" reason="Never"/>
-    <disable_collisions link1="left_inner_knuckle" link2="wrist_2_link" reason="Never"/>
-    <disable_collisions link1="left_inner_knuckle" link2="wrist_3_link" reason="Never"/>
-    <disable_collisions link1="left_outer_finger" link2="left_outer_knuckle" reason="Adjacent"/>
-    <disable_collisions link1="left_outer_finger" link2="right_inner_finger" reason="Never"/>
-    <disable_collisions link1="left_outer_finger" link2="right_inner_finger_pad" reason="Never"/>
-    <disable_collisions link1="left_outer_finger" link2="right_inner_knuckle" reason="Never"/>
-    <disable_collisions link1="left_outer_finger" link2="right_outer_finger" reason="Never"/>
-    <disable_collisions link1="left_outer_finger" link2="right_outer_knuckle" reason="Never"/>
-    <disable_collisions link1="left_outer_finger" link2="robotiq_140_base_link" reason="Never"/>
-    <disable_collisions link1="left_outer_finger" link2="ur_to_robotiq_link" reason="Never"/>
-    <disable_collisions link1="left_outer_finger" link2="wrist_1_link" reason="Never"/>
-    <disable_collisions link1="left_outer_finger" link2="wrist_2_link" reason="Never"/>
-    <disable_collisions link1="left_outer_finger" link2="wrist_3_link" reason="Never"/>
-    <disable_collisions link1="left_outer_knuckle" link2="right_inner_finger" reason="Never"/>
-    <disable_collisions link1="left_outer_knuckle" link2="right_inner_finger_pad" reason="Never"/>
-    <disable_collisions link1="left_outer_knuckle" link2="right_inner_knuckle" reason="Never"/>
-    <disable_collisions link1="left_outer_knuckle" link2="right_outer_finger" reason="Never"/>
-    <disable_collisions link1="left_outer_knuckle" link2="right_outer_knuckle" reason="Never"/>
-    <disable_collisions link1="left_outer_knuckle" link2="robotiq_140_base_link" reason="Adjacent"/>
-    <disable_collisions link1="left_outer_knuckle" link2="ur_to_robotiq_link" reason="Never"/>
-    <disable_collisions link1="left_outer_knuckle" link2="wrist_1_link" reason="Never"/>
-    <disable_collisions link1="left_outer_knuckle" link2="wrist_2_link" reason="Never"/>
-    <disable_collisions link1="left_outer_knuckle" link2="wrist_3_link" reason="Never"/>
-    <disable_collisions link1="right_inner_finger" link2="right_inner_finger_pad" reason="Adjacent"/>
-    <disable_collisions link1="right_inner_finger" link2="right_inner_knuckle" reason="Default"/>
-    <disable_collisions link1="right_inner_finger" link2="right_outer_finger" reason="Adjacent"/>
-    <disable_collisions link1="right_inner_finger" link2="right_outer_knuckle" reason="Never"/>
-    <disable_collisions link1="right_inner_finger" link2="robotiq_140_base_link" reason="Never"/>
-    <disable_collisions link1="right_inner_finger" link2="ur_to_robotiq_link" reason="Never"/>
-    <disable_collisions link1="right_inner_finger" link2="wrist_1_link" reason="Never"/>
-    <disable_collisions link1="right_inner_finger" link2="wrist_2_link" reason="Never"/>
-    <disable_collisions link1="right_inner_finger" link2="wrist_3_link" reason="Never"/>
-    <disable_collisions link1="right_inner_finger_pad" link2="right_inner_knuckle" reason="Never"/>
-    <disable_collisions link1="right_inner_finger_pad" link2="right_outer_finger" reason="Never"/>
-    <disable_collisions link1="right_inner_finger_pad" link2="right_outer_knuckle" reason="Never"/>
-    <disable_collisions link1="right_inner_finger_pad" link2="robotiq_140_base_link" reason="Never"/>
-    <disable_collisions link1="right_inner_finger_pad" link2="ur_to_robotiq_link" reason="Never"/>
-    <disable_collisions link1="right_inner_finger_pad" link2="wrist_1_link" reason="Never"/>
-    <disable_collisions link1="right_inner_finger_pad" link2="wrist_2_link" reason="Never"/>
-    <disable_collisions link1="right_inner_finger_pad" link2="wrist_3_link" reason="Never"/>
-    <disable_collisions link1="right_inner_knuckle" link2="right_outer_finger" reason="Never"/>
-    <disable_collisions link1="right_inner_knuckle" link2="right_outer_knuckle" reason="Default"/>
-    <disable_collisions link1="right_inner_knuckle" link2="robotiq_140_base_link" reason="Adjacent"/>
-    <disable_collisions link1="right_inner_knuckle" link2="ur_to_robotiq_link" reason="Never"/>
-    <disable_collisions link1="right_inner_knuckle" link2="wrist_1_link" reason="Never"/>
-    <disable_collisions link1="right_inner_knuckle" link2="wrist_2_link" reason="Never"/>
-    <disable_collisions link1="right_inner_knuckle" link2="wrist_3_link" reason="Never"/>
-    <disable_collisions link1="right_outer_finger" link2="right_outer_knuckle" reason="Adjacent"/>
-    <disable_collisions link1="right_outer_finger" link2="robotiq_140_base_link" reason="Never"/>
-    <disable_collisions link1="right_outer_finger" link2="ur_to_robotiq_link" reason="Never"/>
-    <disable_collisions link1="right_outer_finger" link2="wrist_1_link" reason="Never"/>
-    <disable_collisions link1="right_outer_finger" link2="wrist_2_link" reason="Never"/>
-    <disable_collisions link1="right_outer_finger" link2="wrist_3_link" reason="Never"/>
-    <disable_collisions link1="right_outer_knuckle" link2="robotiq_140_base_link" reason="Adjacent"/>
-    <disable_collisions link1="right_outer_knuckle" link2="ur_to_robotiq_link" reason="Never"/>
-    <disable_collisions link1="right_outer_knuckle" link2="wrist_1_link" reason="Never"/>
-    <disable_collisions link1="right_outer_knuckle" link2="wrist_2_link" reason="Never"/>
-    <disable_collisions link1="right_outer_knuckle" link2="wrist_3_link" reason="Never"/>
-    <disable_collisions link1="robotiq_140_base_link" link2="ur_to_robotiq_link" reason="Adjacent"/>
-    <disable_collisions link1="robotiq_140_base_link" link2="wrist_1_link" reason="Never"/>
-    <disable_collisions link1="robotiq_140_base_link" link2="wrist_2_link" reason="Never"/>
-    <disable_collisions link1="robotiq_140_base_link" link2="wrist_3_link" reason="Never"/>
-    <disable_collisions link1="shoulder_link" link2="upper_arm_link" reason="Adjacent"/>
-    <disable_collisions link1="shoulder_link" link2="wrist_1_link" reason="Never"/>
-    <disable_collisions link1="ur_to_robotiq_link" link2="wrist_1_link" reason="Never"/>
-    <disable_collisions link1="ur_to_robotiq_link" link2="wrist_2_link" reason="Never"/>
-    <disable_collisions link1="ur_to_robotiq_link" link2="wrist_3_link" reason="Adjacent"/>
-    <disable_collisions link1="wrist_1_link" link2="wrist_2_link" reason="Adjacent"/>
-    <disable_collisions link1="wrist_1_link" link2="wrist_3_link" reason="Never"/>
-    <disable_collisions link1="wrist_2_link" link2="wrist_3_link" reason="Adjacent"/>
+    <disable_collisions link1="${prefix}base_link_inertia" link2="${prefix}shoulder_link" reason="Adjacent"/>
+    <disable_collisions link1="${prefix}base_link_inertia" link2="${prefix}upper_arm_link" reason="Never"/>
+    <disable_collisions link1="${prefix}base_link_inertia" link2="${prefix}wrist_1_link" reason="Never"/>
+    <disable_collisions link1="${prefix}forearm_link" link2="${prefix}upper_arm_link" reason="Adjacent"/>
+    <disable_collisions link1="${prefix}forearm_link" link2="${prefix}wrist_1_link" reason="Adjacent"/>
+    <disable_collisions link1="${prefix}left_inner_finger" link2="${prefix}left_inner_finger_pad" reason="Adjacent"/>
+    <disable_collisions link1="${prefix}left_inner_finger" link2="${prefix}left_inner_knuckle" reason="Default"/>
+    <disable_collisions link1="${prefix}left_inner_finger" link2="${prefix}left_outer_finger" reason="Adjacent"/>
+    <disable_collisions link1="${prefix}left_inner_finger" link2="${prefix}left_outer_knuckle" reason="Never"/>
+    <disable_collisions link1="${prefix}left_inner_finger" link2="${prefix}right_inner_finger" reason="Never"/>
+    <disable_collisions link1="${prefix}left_inner_finger" link2="${prefix}right_inner_finger_pad" reason="Never"/>
+    <disable_collisions link1="${prefix}left_inner_finger" link2="${prefix}right_inner_knuckle" reason="Never"/>
+    <disable_collisions link1="${prefix}left_inner_finger" link2="${prefix}right_outer_finger" reason="Never"/>
+    <disable_collisions link1="${prefix}left_inner_finger" link2="${prefix}right_outer_knuckle" reason="Never"/>
+    <disable_collisions link1="${prefix}left_inner_finger" link2="${prefix}robotiq_140_base_link" reason="Never"/>
+    <disable_collisions link1="${prefix}left_inner_finger" link2="${prefix}ur_to_robotiq_link" reason="Never"/>
+    <disable_collisions link1="${prefix}left_inner_finger" link2="${prefix}wrist_1_link" reason="Never"/>
+    <disable_collisions link1="${prefix}left_inner_finger" link2="${prefix}wrist_2_link" reason="Never"/>
+    <disable_collisions link1="${prefix}left_inner_finger" link2="${prefix}wrist_3_link" reason="Never"/>
+    <disable_collisions link1="${prefix}left_inner_finger_pad" link2="${prefix}left_inner_knuckle" reason="Never"/>
+    <disable_collisions link1="${prefix}left_inner_finger_pad" link2="${prefix}left_outer_finger" reason="Never"/>
+    <disable_collisions link1="${prefix}left_inner_finger_pad" link2="${prefix}left_outer_knuckle" reason="Never"/>
+    <disable_collisions link1="${prefix}left_inner_finger_pad" link2="${prefix}right_inner_finger" reason="Never"/>
+    <disable_collisions link1="${prefix}left_inner_finger_pad" link2="${prefix}right_inner_knuckle" reason="Never"/>
+    <disable_collisions link1="${prefix}left_inner_finger_pad" link2="${prefix}right_outer_finger" reason="Never"/>
+    <disable_collisions link1="${prefix}left_inner_finger_pad" link2="${prefix}right_outer_knuckle" reason="Never"/>
+    <disable_collisions link1="${prefix}left_inner_finger_pad" link2="${prefix}robotiq_140_base_link" reason="Never"/>
+    <disable_collisions link1="${prefix}left_inner_finger_pad" link2="${prefix}ur_to_robotiq_link" reason="Never"/>
+    <disable_collisions link1="${prefix}left_inner_finger_pad" link2="${prefix}wrist_1_link" reason="Never"/>
+    <disable_collisions link1="${prefix}left_inner_finger_pad" link2="${prefix}wrist_2_link" reason="Never"/>
+    <disable_collisions link1="${prefix}left_inner_finger_pad" link2="${prefix}wrist_3_link" reason="Never"/>
+    <disable_collisions link1="${prefix}left_inner_knuckle" link2="${prefix}left_outer_finger" reason="Never"/>
+    <disable_collisions link1="${prefix}left_inner_knuckle" link2="${prefix}left_outer_knuckle" reason="Default"/>
+    <disable_collisions link1="${prefix}left_inner_knuckle" link2="${prefix}right_inner_finger" reason="Never"/>
+    <disable_collisions link1="${prefix}left_inner_knuckle" link2="${prefix}right_inner_finger_pad" reason="Never"/>
+    <disable_collisions link1="${prefix}left_inner_knuckle" link2="${prefix}right_inner_knuckle" reason="Never"/>
+    <disable_collisions link1="${prefix}left_inner_knuckle" link2="${prefix}right_outer_finger" reason="Never"/>
+    <disable_collisions link1="${prefix}left_inner_knuckle" link2="${prefix}right_outer_knuckle" reason="Never"/>
+    <disable_collisions link1="${prefix}left_inner_knuckle" link2="${prefix}robotiq_140_base_link" reason="Adjacent"/>
+    <disable_collisions link1="${prefix}left_inner_knuckle" link2="${prefix}ur_to_robotiq_link" reason="Never"/>
+    <disable_collisions link1="${prefix}left_inner_knuckle" link2="${prefix}wrist_1_link" reason="Never"/>
+    <disable_collisions link1="${prefix}left_inner_knuckle" link2="${prefix}wrist_2_link" reason="Never"/>
+    <disable_collisions link1="${prefix}left_inner_knuckle" link2="${prefix}wrist_3_link" reason="Never"/>
+    <disable_collisions link1="${prefix}left_outer_finger" link2="${prefix}left_outer_knuckle" reason="Adjacent"/>
+    <disable_collisions link1="${prefix}left_outer_finger" link2="${prefix}right_inner_finger" reason="Never"/>
+    <disable_collisions link1="${prefix}left_outer_finger" link2="${prefix}right_inner_finger_pad" reason="Never"/>
+    <disable_collisions link1="${prefix}left_outer_finger" link2="${prefix}right_inner_knuckle" reason="Never"/>
+    <disable_collisions link1="${prefix}left_outer_finger" link2="${prefix}right_outer_finger" reason="Never"/>
+    <disable_collisions link1="${prefix}left_outer_finger" link2="${prefix}right_outer_knuckle" reason="Never"/>
+    <disable_collisions link1="${prefix}left_outer_finger" link2="${prefix}robotiq_140_base_link" reason="Never"/>
+    <disable_collisions link1="${prefix}left_outer_finger" link2="${prefix}ur_to_robotiq_link" reason="Never"/>
+    <disable_collisions link1="${prefix}left_outer_finger" link2="${prefix}wrist_1_link" reason="Never"/>
+    <disable_collisions link1="${prefix}left_outer_finger" link2="${prefix}wrist_2_link" reason="Never"/>
+    <disable_collisions link1="${prefix}left_outer_finger" link2="${prefix}wrist_3_link" reason="Never"/>
+    <disable_collisions link1="${prefix}left_outer_knuckle" link2="${prefix}right_inner_finger" reason="Never"/>
+    <disable_collisions link1="${prefix}left_outer_knuckle" link2="${prefix}right_inner_finger_pad" reason="Never"/>
+    <disable_collisions link1="${prefix}left_outer_knuckle" link2="${prefix}right_inner_knuckle" reason="Never"/>
+    <disable_collisions link1="${prefix}left_outer_knuckle" link2="${prefix}right_outer_finger" reason="Never"/>
+    <disable_collisions link1="${prefix}left_outer_knuckle" link2="${prefix}right_outer_knuckle" reason="Never"/>
+    <disable_collisions link1="${prefix}left_outer_knuckle" link2="${prefix}robotiq_140_base_link" reason="Adjacent"/>
+    <disable_collisions link1="${prefix}left_outer_knuckle" link2="${prefix}ur_to_robotiq_link" reason="Never"/>
+    <disable_collisions link1="${prefix}left_outer_knuckle" link2="${prefix}wrist_1_link" reason="Never"/>
+    <disable_collisions link1="${prefix}left_outer_knuckle" link2="${prefix}wrist_2_link" reason="Never"/>
+    <disable_collisions link1="${prefix}left_outer_knuckle" link2="${prefix}wrist_3_link" reason="Never"/>
+    <disable_collisions link1="${prefix}right_inner_finger" link2="${prefix}right_inner_finger_pad" reason="Adjacent"/>
+    <disable_collisions link1="${prefix}right_inner_finger" link2="${prefix}right_inner_knuckle" reason="Default"/>
+    <disable_collisions link1="${prefix}right_inner_finger" link2="${prefix}right_outer_finger" reason="Adjacent"/>
+    <disable_collisions link1="${prefix}right_inner_finger" link2="${prefix}right_outer_knuckle" reason="Never"/>
+    <disable_collisions link1="${prefix}right_inner_finger" link2="${prefix}robotiq_140_base_link" reason="Never"/>
+    <disable_collisions link1="${prefix}right_inner_finger" link2="${prefix}ur_to_robotiq_link" reason="Never"/>
+    <disable_collisions link1="${prefix}right_inner_finger" link2="${prefix}wrist_1_link" reason="Never"/>
+    <disable_collisions link1="${prefix}right_inner_finger" link2="${prefix}wrist_2_link" reason="Never"/>
+    <disable_collisions link1="${prefix}right_inner_finger" link2="${prefix}wrist_3_link" reason="Never"/>
+    <disable_collisions link1="${prefix}right_inner_finger_pad" link2="${prefix}right_inner_knuckle" reason="Never"/>
+    <disable_collisions link1="${prefix}right_inner_finger_pad" link2="${prefix}right_outer_finger" reason="Never"/>
+    <disable_collisions link1="${prefix}right_inner_finger_pad" link2="${prefix}right_outer_knuckle" reason="Never"/>
+    <disable_collisions link1="${prefix}right_inner_finger_pad" link2="${prefix}robotiq_140_base_link" reason="Never"/>
+    <disable_collisions link1="${prefix}right_inner_finger_pad" link2="${prefix}ur_to_robotiq_link" reason="Never"/>
+    <disable_collisions link1="${prefix}right_inner_finger_pad" link2="${prefix}wrist_1_link" reason="Never"/>
+    <disable_collisions link1="${prefix}right_inner_finger_pad" link2="${prefix}wrist_2_link" reason="Never"/>
+    <disable_collisions link1="${prefix}right_inner_finger_pad" link2="${prefix}wrist_3_link" reason="Never"/>
+    <disable_collisions link1="${prefix}right_inner_knuckle" link2="${prefix}right_outer_finger" reason="Never"/>
+    <disable_collisions link1="${prefix}right_inner_knuckle" link2="${prefix}right_outer_knuckle" reason="Default"/>
+    <disable_collisions link1="${prefix}right_inner_knuckle" link2="${prefix}robotiq_140_base_link" reason="Adjacent"/>
+    <disable_collisions link1="${prefix}right_inner_knuckle" link2="${prefix}ur_to_robotiq_link" reason="Never"/>
+    <disable_collisions link1="${prefix}right_inner_knuckle" link2="${prefix}wrist_1_link" reason="Never"/>
+    <disable_collisions link1="${prefix}right_inner_knuckle" link2="${prefix}wrist_2_link" reason="Never"/>
+    <disable_collisions link1="${prefix}right_inner_knuckle" link2="${prefix}wrist_3_link" reason="Never"/>
+    <disable_collisions link1="${prefix}right_outer_finger" link2="${prefix}right_outer_knuckle" reason="Adjacent"/>
+    <disable_collisions link1="${prefix}right_outer_finger" link2="${prefix}robotiq_140_base_link" reason="Never"/>
+    <disable_collisions link1="${prefix}right_outer_finger" link2="${prefix}ur_to_robotiq_link" reason="Never"/>
+    <disable_collisions link1="${prefix}right_outer_finger" link2="${prefix}wrist_1_link" reason="Never"/>
+    <disable_collisions link1="${prefix}right_outer_finger" link2="${prefix}wrist_2_link" reason="Never"/>
+    <disable_collisions link1="${prefix}right_outer_finger" link2="${prefix}wrist_3_link" reason="Never"/>
+    <disable_collisions link1="${prefix}right_outer_knuckle" link2="${prefix}robotiq_140_base_link" reason="Adjacent"/>
+    <disable_collisions link1="${prefix}right_outer_knuckle" link2="${prefix}ur_to_robotiq_link" reason="Never"/>
+    <disable_collisions link1="${prefix}right_outer_knuckle" link2="${prefix}wrist_1_link" reason="Never"/>
+    <disable_collisions link1="${prefix}right_outer_knuckle" link2="${prefix}wrist_2_link" reason="Never"/>
+    <disable_collisions link1="${prefix}right_outer_knuckle" link2="${prefix}wrist_3_link" reason="Never"/>
+    <disable_collisions link1="${prefix}robotiq_140_base_link" link2="${prefix}ur_to_robotiq_link" reason="Adjacent"/>
+    <disable_collisions link1="${prefix}robotiq_140_base_link" link2="${prefix}wrist_1_link" reason="Never"/>
+    <disable_collisions link1="${prefix}robotiq_140_base_link" link2="${prefix}wrist_2_link" reason="Never"/>
+    <disable_collisions link1="${prefix}robotiq_140_base_link" link2="${prefix}wrist_3_link" reason="Never"/>
+    <disable_collisions link1="${prefix}shoulder_link" link2="${prefix}upper_arm_link" reason="Adjacent"/>
+    <disable_collisions link1="${prefix}shoulder_link" link2="${prefix}wrist_1_link" reason="Never"/>
+    <disable_collisions link1="${prefix}ur_to_robotiq_link" link2="${prefix}wrist_1_link" reason="Never"/>
+    <disable_collisions link1="${prefix}ur_to_robotiq_link" link2="${prefix}wrist_2_link" reason="Never"/>
+    <disable_collisions link1="${prefix}ur_to_robotiq_link" link2="${prefix}wrist_3_link" reason="Adjacent"/>
+    <disable_collisions link1="${prefix}wrist_1_link" link2="${prefix}wrist_2_link" reason="Adjacent"/>
+    <disable_collisions link1="${prefix}wrist_1_link" link2="${prefix}wrist_3_link" reason="Never"/>
+    <disable_collisions link1="${prefix}wrist_2_link" link2="${prefix}wrist_3_link" reason="Adjacent"/>
+    <xacro:if value="${use_cam_flange_support}">
+      <xacro:include filename="$(find cam_flange_support)/srdf/cam_flange_support_collisions_macro.srdf.xacro"/>
+      <xacro:cam_flange_support_collisions
+        prefix="${prefix}"
+        parent_1="${prefix}tool0"
+        child_1="${prefix}ur_to_robotiq_link"
+      />
+    </xacro:if>
   </xacro:macro>
 </robot>
