Commit message: Stand, auxiliary table, and L aluminum profile included in urdf (with launch argument)

File: setup_description/urdf/robot.urdf.xacro (robot description, xacro)
@@ -3,4 +3,5 @@
   <xacro:arg name="name" default="ur"/>
   <xacro:arg name="use_sim" default="false"/>
+  <xacro:arg name="include_digilab" default="false"/>
   <xacro:include filename="$(find ur_description)/urdf/ur_macro.xacro"/>
   <xacro:include filename="$(find robotiq_description)/urdf/robotiq_2f_140_macro.urdf.xacro" />
@@ -45,9 +46,21 @@
   <!-- create link fixed to the "world" -->
   <link name="world" />
+  <!-- Digilab -->
+  <xacro:property name="comparable_include_digilab" value="$(arg include_digilab)" />
+  <xacro:if value="${comparable_include_digilab}">
+    <xacro:include filename="$(find setup_description)/urdf/digilab_macro.urdf.xacro" />
+    <xacro:digilab parent="world" prefix="">
+      <origin xyz="0 0 0" rpy="0 0 0"/>
+    </xacro:digilab>
+    <xacro:property name="ur_parent" value="stand_mounting" />
+  </xacro:if>
+  <xacro:unless value="${comparable_include_digilab}">
+    <xacro:property name="ur_parent" value="world" />
+  </xacro:unless>
   <!-- arm -->
   <xacro:ur_robot
     name="$(arg name)"
     tf_prefix="$(arg tf_prefix)"
-    parent="world"
+    parent="${ur_parent}"
     joint_limits_parameters_file="$(arg joint_limit_params)"
     kinematics_parameters_file="$(arg kinematics_params)"

Commit message: Visualization working

File: setup_description/urdf/robot.urdf.xacro (robot description, xacro)
@@ -131,5 +131,12 @@
   <!-- Realsense D435 Camera -->
   <xacro:sensor_d435 parent="base_link" use_nominal_extrinsics="$(arg use_nominal_extrinsics)" add_plug="$(arg add_plug)" use_mesh="$(arg use_mesh)">
-    <origin xyz="0 0 1.0" rpy="0 0 0"/>
+    <origin xyz="-1.209944 0.231354 0.232905" rpy="0.002605 0.729241 0.762238"/>
   </xacro:sensor_d435>
+  <!-- Calibration Frame-->
+  <link name="charuco_board"/>
+  <joint name="charuco_board_joint" type="fixed">
+    <parent link="robotiq_base_link"/>
+    <child link="charuco_board"/>
+    <origin xyz="-0.15 0 0.15" rpy="0 0 -1.5708"/>
+  </joint>
 </robot>

Commit message: Working routine

File: setup_description/urdf/robot.urdf.xacro (robot description, xacro)
@@ -95,5 +95,5 @@
     <xacro:include filename="$(find cam_flange_support)/urdf/cam_flange_support_macro.urdf.xacro" />
     <xacro:cam_flange_support parent="tool0" >
-      <origin xyz="0 0 0" rpy="0 0 ${pi}" />
+      <origin xyz="0 0 0" rpy="0 0 0" />
     </xacro:cam_flange_support>
   </xacro:if>
@@ -131,6 +131,7 @@
   <!-- Realsense D435 Camera -->
   <xacro:sensor_d435 parent="base_link" use_nominal_extrinsics="$(arg use_nominal_extrinsics)" add_plug="$(arg add_plug)" use_mesh="$(arg use_mesh)">
-    <origin xyz="-1.209944 0.231354 0.232905" rpy="0.002605 0.729241 0.762238"/>
+    <origin xyz="-1.090329 0.318755 0.635220" rpy="-0.015609 0.316050 0.494161"/>
   </xacro:sensor_d435>
+  <!-- ADDITIONAL FRAMES -->
   <!-- Calibration Frame-->
   <link name="charuco_board"/>
@@ -140,3 +141,10 @@
     <origin xyz="-0.15 0 0.15" rpy="0 0 -1.5708"/>
   </joint>
+  <!-- Place Frame -->
+  <link name="object_place"/>
+  <joint name="object_place_joint" type="fixed">
+    <parent link="world"/>
+    <child link="object_place"/>
+    <origin xyz="-0.220 0.587 0.152" rpy="-3.083 0.018 -1.727"/>
+  </joint>
 </robot>

File: setup_moveit_config/srdf/ur_macro.srdf.xacro (robot description, xacro)
@@ -40,10 +40,10 @@
     </group_state>
     <group_state name="${prefix}observation" group="${prefix}${name}_manipulator">
-      <joint name="${prefix}elbow_joint" value="-1.8814754486083984" />
-      <joint name="${prefix}shoulder_lift_joint" value="-1.6091319523253382" />
-      <joint name="${prefix}shoulder_pan_joint" value="6.053856372833252" />
-      <joint name="${prefix}wrist_1_joint" value="-0.9247403305820008" />
-      <joint name="${prefix}wrist_2_joint" value="1.6628847122192383" />
-      <joint name="${prefix}wrist_3_joint" value="2.8549625873565674" />
+      <joint name="${prefix}elbow_joint" value="-1.6927485466003418" />
+      <joint name="${prefix}shoulder_lift_joint" value="-1.4086332035115738" />
+      <joint name="${prefix}shoulder_pan_joint" value="-0.604955021535055" />
+      <joint name="${prefix}wrist_1_joint" value="5.252929734974661" />
+      <joint name="${prefix}wrist_2_joint" value="-4.3677746693240564" />
+      <joint name="${prefix}wrist_3_joint" value="-3.6066013018237513" />
     </group_state>
     <group name="gripper">

Commit message: README update

File: setup_description/urdf/robot.urdf.xacro (robot description, xacro)
@@ -131,5 +131,5 @@
   <!-- Realsense D435 Camera -->
   <xacro:sensor_d435 parent="base_link" use_nominal_extrinsics="$(arg use_nominal_extrinsics)" add_plug="$(arg add_plug)" use_mesh="$(arg use_mesh)">
-    <origin xyz="-1.090329 0.318755 0.635220" rpy="-0.015609 0.316050 0.494161"/>
+    <origin xyz="-1.090329 0.318755 0.635220" rpy="-0.015609 0.316050 0.494161"/> <!-- SET CAMERA EXTRINSICS -->
   </xacro:sensor_d435>
   <!-- ADDITIONAL FRAMES -->
@@ -139,5 +139,5 @@
     <parent link="robotiq_base_link"/>
     <child link="charuco_board"/>
-    <origin xyz="-0.15 0 0.15" rpy="0 0 -1.5708"/>
+    <origin xyz="-0.15 0 0.15" rpy="0 0 -1.5708"/> <!-- SET CALIBRATION BOARD FRAME -->
   </joint>
   <!-- Place Frame -->
@@ -146,5 +146,5 @@
     <parent link="world"/>
     <child link="object_place"/>
-    <origin xyz="-0.220 0.587 0.152" rpy="-3.083 0.018 -1.727"/>
+    <origin xyz="-0.220 0.587 0.152" rpy="-3.083 0.018 -1.727"/> <!-- SET OBJECT PLACE FRAME -->
   </joint>
 </robot>

Commit message: Velocity and acceleration scaling

File: setup_description/urdf/robot.urdf.xacro (robot description, xacro)
@@ -131,5 +131,5 @@
   <!-- Realsense D435 Camera -->
   <xacro:sensor_d435 parent="base_link" use_nominal_extrinsics="$(arg use_nominal_extrinsics)" add_plug="$(arg add_plug)" use_mesh="$(arg use_mesh)">
-    <origin xyz="-1.090329 0.318755 0.635220" rpy="-0.015609 0.316050 0.494161"/> <!-- SET CAMERA EXTRINSICS -->
+    <origin xyz="-1.093909 0.336769 0.632084" rpy="-0.061686 0.315636 0.434503"/> <!-- SET CAMERA EXTRINSICS -->
   </xacro:sensor_d435>
   <!-- ADDITIONAL FRAMES -->

File: setup_moveit_config/srdf/ur_macro.srdf.xacro (robot description, xacro)
@@ -16,10 +16,10 @@
     <!--GROUP STATES - Purpose - Define a named state for a particular group, in terms of joint values. This is useful to define states like 'folded arms'-->
     <group_state name="${prefix}home" group="${prefix}${name}_manipulator">
-      <joint name="${prefix}elbow_joint" value="-2.0100371837615967" />
-      <joint name="${prefix}shoulder_lift_joint" value="-1.104203389292099" />
-      <joint name="${prefix}shoulder_pan_joint" value="4.682784557342529" />
-      <joint name="${prefix}wrist_1_joint" value="-1.4381349843791504" />
-      <joint name="${prefix}wrist_2_joint" value="1.628240942955017" />
-      <joint name="${prefix}wrist_3_joint" value="3.2838845252990723" />
+      <joint name="${prefix}elbow_joint" value="-1.972432017326355" />
+      <joint name="${prefix}shoulder_lift_joint" value="-0.8492182058146973" />
+      <joint name="${prefix}shoulder_pan_joint" value="-1.3801501433001917" />
+      <joint name="${prefix}wrist_1_joint" value="4.819335925370016" />
+      <joint name="${prefix}wrist_2_joint" value="-4.822485152875082" />
+      <joint name="${prefix}wrist_3_joint" value="-2.948768440877096" />
     </group_state>
     <group_state name="${prefix}up" group="${prefix}${name}_manipulator">
